File: station/eda/WeatherStation.sch (EAGLE design)
At the start: 15 parts, among them IC1 ESP-12E/F

Commit message: update for rev B
Parts:
- R1, R3: value 7.5K -> 6K8
Changed lines of the file:
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@@
 <part name="SUPPLY1" library="Tutorial - Fusion 360" deviceset="GND" device=""/>
 <part name="R2" library="Resistor" deviceset="R-US" device="CHIP-0805(2012-METRIC)" package3d_urn="urn:adsk.eagle:package:16378559/2" technology="_" value="10K"/>
-<part name="R1" library="Resistor" deviceset="R-US" device="CHIP-0805(2012-METRIC)" package3d_urn="urn:adsk.eagle:package:16378559/2" technology="_" value="7.5K"/>
-<part name="R3" library="Resistor" deviceset="R-US" device="CHIP-0805(2012-METRIC)" package3d_urn="urn:adsk.eagle:package:16378559/2" technology="_" value="7.5K"/>
+<part name="R1" library="Resistor" deviceset="R-US" device="CHIP-0805(2012-METRIC)" package3d_urn="urn:adsk.eagle:package:16378559/2" technology="_" value="6K8"/>
+<part name="R3" library="Resistor" deviceset="R-US" device="CHIP-0805(2012-METRIC)" package3d_urn="urn:adsk.eagle:package:16378559/2" technology="_" value="6K8"/>
 <part name="SUPPLY5" library="Tutorial - Fusion 360" deviceset="GND" device=""/>
 <part name="SUPPLY6" library="Tutorial - Fusion 360" deviceset="GND" device=""/>
