File: station/eda/WeatherStationPCB.brd (EAGLE design)
At the start: 53 x 25 mm, 15 parts, among them IC1 ESP-12E/F

Commit message: update for rev B
Parts:
- R1, R3: value 7.5K -> 6K8
Routing:
- net GND: track 101.2 -> 20.6 mm, vias 0 -> 3
- net +3.3V: track 93.4 -> 35.5 mm
- added copper zone on layer 1, net +3.3V
- added copper zone on layer 16, net GND
Other:
- board text added: "Revision B"
- board text added: "Solar Wx Station Rev. B"
- board text added: "github.com/mmangus/wxmon"
- board text removed: "Revision A"
- board text removed: "Solar Wx Station Rev. A"
- board text removed: "github.com/mmangus/wxsta"
